Commit message: fixed prefix issue

File: urdf/sensor_imu.xacro (robot description, xacro)
@@ -2,8 +2,7 @@
 <robot xmlns:sensor="http://playerstage.sourceforge.net/gazebo/xmlschema/#sensor" xmlns:controller="http://playerstage.sourceforge.net/gazebo/xmlschema/#controller" xmlns:interface="http://playerstage.sourceforge.net/gazebo/xmlschema/#interface" xmlns:xacro="http://ros.org/wiki/xacro" name="sensor_imu">
       iption)/urdf/base/as_base.macro.xacro" />
-      <xacro:arg name="prefix" default="sensor" />
       <xacro:property name="sensor_xyz" value=" 0.007 0 0" />
       <xacro:property name="sensor_rpy" value="0 0 0" />
-      <xacro:macro name="imu" params="prefix:='' parent:='base_link' rpy:='0 0 0' xyz:='0 0 0'">
+      <xacro:macro name="imu" params="prefix:='' ns:='as_sensors' parent:='base_link' rpy:='0 0 0' xyz:='0 0 0'">
             <joint name="${prefix}_imu_module_joint1" type="fixed">
                   <parent link="${parent}" />
@@ -28,7 +27,7 @@
                         <alwaysOn>true</alwaysOn>
                         <bodyName>${prefix}_imu_frame</bodyName>
-                        <topicName>${prefix}_imu</topicName>
-                        <serviceName>${prefix}_imu_service</serviceName>
-                        <gaussianNoise>0.03</gaussianNoise>
+                        <topicName>${ns}/${prefix}_imu</topicName>
+                        <serviceName>${ns}/${prefix}_imu_service</serviceName>
+                        <gaussianNoise>0.32</gaussianNoise>
                         <updateRate>100.0</updateRate>
                   </plugin>
